Commit message: Added Module_2

File: src/ros2_packages/humanoid_control/urdf/basic_humanoid.urdf (robot description, URDF)
Before this commit: robot basic_humanoid, 15 links, 14 joints
Links:
- added link camera_link, mass 0.01; collision box size=0.02 0.04 0.02; visual box size=0.02 0.04 0.02
- added link lidar_link, mass 0.1; collision cylinder length=0.05 radius=0.02; visual cylinder length=0.05 radius=0.02
Joints:
- added joint camera_joint: type fixed, parent head, child camera_link, origin xyz=0.09 0 0.02 rpy=0 0 0
- added joint lidar_joint: type fixed, parent head, child lidar_link, origin xyz=0.08 0 0 rpy=0 0 0
